Commit message: fix: move camera_link from chassis to arm_yanthra_link

File: pragati_ros2/src/vehicle_arm_sim/urdf/saved/vehicle_arm_merged.urdf (robot description, URDF)
Before this commit: robot vehicle_arm, 54 links, 53 joints
Joints:
- joint camera_joint: origin xyz=1.55 -0.25 0.9 rpy=-1.5707963267948966 0.0 -0.2618 -> xyz=0.016845 0.100461 -0.077129 rpy=1.5708 0.785398 0; parent base-v1 -> arm_yanthra_link

File: pragati_ros2/src/vehicle_arm_sim/urdf/vehicle_arm_merged.urdf (robot description, URDF)
Before this commit: robot vehicle_arm, 54 links, 53 joints
Joints:
- joint camera_joint: origin xyz=1.55 -0.25 0.9 rpy=-1.5707963267948966 0.0 -0.2618 -> xyz=0.016845 0.100461 -0.077129 rpy=1.5708 0.785398 0; parent base-v1 -> arm_yanthra_link
